File: PCBs/mainPCB/mainPCB.kicad_pcb (KiCad board)
At the start: 2 copper layers, 80 x 100.5 mm, 9 parts, among them SW1 RotaryEncoder_Switch, SW2 SW_Push, SW3 SW_Push, SW4 SW_Push

Commit message: fixed PCB
retraced few traces, reworked rotary encoder to completely different design
Parts:
- removed SW1: RotaryEncoder_Switch, Rotary_Encoder:RotaryEncoder_Alps_EC11E-Switch_Vertical_H20mm_CircularMountingHoles
- added U1: KY-040, KY-040:KY-040-PORT, F.Cu at (150.2, 130.5)
Connections:
- A1 pad 40: unconnected-(A1-VBUS-Pad40) -> Net-(A1-VBUS)
Routing:
- net Net-(A1-VBUS): track 0.00 -> 106.7 mm
- net Net-(A1-GPIO18): track 64.6 -> 39.4 mm
- net Net-(A1-GPIO16): track 34.5 -> 42.2 mm
- net Net-(A1-GPIO17): track 35.1 -> 40.9 mm

Commit message: small fixes for PCB
Parts:
- moved H3 12.6 mm to (100.0, 140.0)
- moved H4 10.5 mm to (160.5, 140.0)
- moved H2 7.00 mm to (100.0, 60.0)
Other:
- board size 80 x 100.5 mm -> 69 x 88.5 mm
Changed lines of the file:
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@@
 	(footprint "MountingHole:MountingHole_3.2mm_M3_DIN965"
 		(layer "F.Cu")
-		(at 93 60)
+		(at 100 60)
 		(descr "Mounting Hole 3.2mm, M3, no annular, generated by kicad-footprint-generator mountinghole.py")
 		(tags "mountinghole M3 DIN965")
@@
 	(footprint "MountingHole:MountingHole_3.2mm_M3_DIN965"
 		(layer "F.Cu")
-		(at 93 150.5)
+		(at 100 140)
 		(descr "Mounting Hole 3.2mm, M3, no annular, generated by kicad-footprint-generator mountinghole.py")
 		(tags "mountinghole M3 DIN965")
@@
 	(footprint "MountingHole:MountingHole_3.2mm_M3_DIN965"
 		(layer "F.Cu")
-		(at 160.5 150.5)
+		(at 160.5 140)
 		(descr "Mounting Hole 3.2mm, M3, no annular, generated by kicad-footprint-generator mountinghole.py")
 		(tags "mountinghole M3 DIN965")
@@
 	)
 	(gr_rect
-		(start 86.5 54.75)
-		(end 166.5 155.25)
+		(start 95.5 55.5)
+		(end 164.5 144)
 		(stroke
 			(width 0.05)
@@
 	)
 	(segment
-		(start 147.09 105.47)
-		(end 123.19 105.47)
-		(width 0.2)
-		(layer "F.Cu")
-		(net "Net-(A1-GPIO19)")
-	)
-	(segment
-		(start 151.54 109.92)
-		(end 147.09 105.47)
-		(width 0.2)
-		(layer "F.Cu")
-		(net "Net-(A1-GPIO19)")
-	)
-	(segment
-		(start 131.5 119)
-		(end 128.13 115.63)
-		(width 0.2)
-		(layer "F.Cu")
-		(net "Net-(A1-GPIO16)")
-	)
-	(segment
-		(start 131.5 126.5)
-		(end 131.5 119)
-		(width 0.2)
-		(layer "F.Cu")
-		(net "Net-(A1-GPIO16)")
-	)
-	(segment
-		(start 128.13 115.63)
-		(end 123.19 115.63)
+		(start 137.51 108.01)
+		(end 123.19 108.01)
 		(width 0.2)
 		(layer "F.Cu")
-		(net "Net-(A1-GPIO16)")
+		(net "Net-(A1-GPIO18)")
 	)
 	(segment
-		(start 144.5 136.5)
-		(end 141.5 136.5)
+		(start 143.8462 125.3462)
+		(end 139 120.5)
 		(width 0.2)
 		(layer "F.Cu")
-		(net "Net-(A1-GPIO16)")
+		(net "Net-(A1-GPIO18)")
 	)
 	(segment
-		(start 141.5 136.5)
-		(end 131.5 126.5)
+		(start 139 109.5)
+		(end 137.51 108.01)
 		(width 0.2)
 		(layer "F.Cu")
-		(net "Net-(A1-GPIO16)")
+		(net "Net-(A1-GPIO18)")
 	)
 	(segment
-		(start 148.9262 130.5)
-		(end 148.9262 132.0738)
+		(start 143.8462 130.5)
+		(end 143.8462 125.3462)
 		(width 0.2)
 		(layer "F.Cu")
-		(net "Net-(A1-GPIO16)")
+		(net "Net-(A1-GPIO18)")
 	)
 	(segment
-		(start 148.9262 132.0738)
-		(end 144.5 136.5)
+		(start 139 120.5)
+		(end 139 109.5)
 		(width 0.2)
 		(layer "F.Cu")
-		(net "Net-(A1-GPIO16)")
+		(net "Net-(A1-GPIO18)")
 	)
 	(segment
@@
 	)
 	(segment
-		(start 137.51 108.01)
-		(end 123.19 108.01)
-		(width 0.2)
-		(layer "F.Cu")
-		(net "Net-(A1-GPIO18)")
-	)
-	(segment
-		(start 143.8462 125.3462)
-		(end 139 120.5)
+		(start 131.5 119)
+		(end 128.13 115.63)
 		(width 0.2)
 		(layer "F.Cu")
-		(net "Net-(A1-GPIO18)")
+		(net "Net-(A1-GPIO16)")
 	)
 	(segment
-		(start 139 109.5)
-		(end 137.51 108.01)
+		(start 131.5 126.5)
+		(end 131.5 119)
 		(width 0.2)
 		(layer "F.Cu")
-		(net "Net-(A1-GPIO18)")
+		(net "Net-(A1-GPIO16)")
 	)
 	(segment
-		(start 143.8462 130.5)
-		(end 143.8462 125.3462)
+		(start 128.13 115.63)
+		(end 123.19 115.63)
 		(width 0.2)
 		(layer "F.Cu")
-		(net "Net-(A1-GPIO18)")
+		(net "Net-(A1-GPIO16)")
 	)
 	(segment
-		(start 139 120.5)
-		(end 139 109.5)
+		(start 144.5 136.5)
+		(end 141.5 136.5)
 		(width 0.2)
 		(layer "F.Cu")
-		(net "Net-(A1-GPIO18)")
+		(net "Net-(A1-GPIO16)")
 	)
 	(segment
-		(start 128.57 102.93)
-		(end 123.19 102.93)
+		(start 141.5 136.5)
+		(end 131.5 126.5)
 		(width 0.2)
 		(layer "F.Cu")
-		(net "Net-(A1-GPIO20)")
+		(net "Net-(A1-GPIO16)")
 	)
 	(segment
-		(start 141.58 89.92)
-		(end 128.57 102.93)
+		(start 148.9262 130.5)
+		(end 148.9262 132.0738)
 		(width 0.2)
 		(layer "F.Cu")
-		(net "Net-(A1-GPIO20)")
+		(net "Net-(A1-GPIO16)")
 	)
 	(segment
-		(start 151.54 89.92)
-		(end 141.58 89.92)
+		(start 148.9262 132.0738)
+		(end 144.5 136.5)
 		(width 0.2)
 		(layer "F.Cu")
-		(net "Net-(A1-GPIO20)")
+		(net "Net-(A1-GPIO16)")
 	)
 	(segment
@@
 		(net "Net-(A1-VBUS)")
 	)
+	(segment
+		(start 147.09 105.47)
+		(end 123.19 105.47)
+		(width 0.2)
+		(layer "F.Cu")
+		(net "Net-(A1-GPIO19)")
+	)
+	(segment
+		(start 151.54 109.92)
+		(end 147.09 105.47)
+		(width 0.2)
+		(layer "F.Cu")
+		(net "Net-(A1-GPIO19)")
+	)
+	(segment
+		(start 128.57 102.93)
+		(end 123.19 102.93)
+		(width 0.2)
+		(layer "F.Cu")
+		(net "Net-(A1-GPIO20)")
+	)
+	(segment
+		(start 141.58 89.92)
+		(end 128.57 102.93)
+		(width 0.2)
+		(layer "F.Cu")
+		(net "Net-(A1-GPIO20)")
+	)
+	(segment
+		(start 151.54 89.92)
+		(end 141.58 89.92)
+		(width 0.2)
+		(layer "F.Cu")
+		(net "Net-(A1-GPIO20)")
+	)
 	(zone
 		(net "Net-(A1-GND-Pad13)")
@@
 		(polygon
 			(pts
-				(xy 93 60) (xy 93 150.5) (xy 160.5 150.5) (xy 160 60)
+				(xy 100 60) (xy 100 140) (xy 160.441989 140) (xy 160 60)
 			)
 		)

Commit message: CAD
added base plate and lid for macro keyboard container
Parts:
- moved H2 0.50 mm to (100.5, 60.0)
- moved H3 0.50 mm to (100.5, 140.0)
Changed lines of the file:
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@@
 			(outputformat 1)
 			(mirror no)
-			(drillshape 1)
+			(drillshape 0)
 			(scaleselection 1)
-			(outputdirectory "")
+			(outputdirectory "../GRB_PCB/")
 		)
 	)
 	(footprint "MountingHole:MountingHole_3.2mm_M3_DIN965"
 		(layer "F.Cu")
-		(at 100 60)
+		(at 100.5 60)
 		(descr "Mounting Hole 3.2mm, M3, no annular, generated by kicad-footprint-generator mountinghole.py")
 		(tags "mountinghole M3 DIN965")
@@
 	(footprint "MountingHole:MountingHole_3.2mm_M3_DIN965"
 		(layer "F.Cu")
-		(at 100 140)
+		(at 100.5 140)
 		(descr "Mounting Hole 3.2mm, M3, no annular, generated by kicad-footprint-generator mountinghole.py")
 		(tags "mountinghole M3 DIN965")
@@
 		(polygon
 			(pts
-				(xy 100 60) (xy 100 140) (xy 160.441989 140) (xy 160 60)
+				(xy 100.5 60) (xy 100.5 140) (xy 160.441989 140) (xy 160 60)
 			)
 		)
